Commit message: change QoS for dashing API

File: cartographer_ros/urdf/backpack_2d.urdf (robot description, URDF)
Before this commit: robot cartographer_backpack_2d, 4 links, 3 joints
Links:
- removed link horizontal_laser_link
- added link echoes; visual cylinder length=0.05 radius=0.03
Joints:
- joint horizontal_laser_link_joint: child horizontal_laser_link -> echoes
